Commit message: Update files for custom robot

File: frontend/public/urdf/PAROL6.urdf (robot description, URDF)
Before this commit: robot parol6, 8 links, 7 joints
Links:
- link L1: mass 0.644800830530233 -> None; geometry visual mesh filename=./meshes/j1.stl scale=0.01 0.01 0.01
- link L2: mass 0.512334779399788 -> None; geometry visual mesh filename=./meshes/j2.stl scale=0.01 0.01 0.01
- link L3: mass 0.550970997806044 -> None; geometry visual mesh filename=./meshes/j3.stl scale=0.01 0.01 0.01
- link L4: mass 0.39346362633915 -> None; geometry visual mesh filename=./meshes/j4.stl scale=0.01 0.01 0.01
- link L5: mass 0.185171777001718 -> None; geometry visual mesh filename=./meshes/j5.stl scale=0.01 0.01 0.01
- link L6: mass 0.0703261410665101 -> None; geometry 
- link base_link: mass 0.812661291810144 -> None; geometry visual mesh filename=./meshes/base.stl scale=0.01 0.01 0.01
Joints:
- joint L1: limit lower=-2.1475731 upper=2.1475731 effort=300 velocity=3 -> lower=-1.0471975512 upper=1.0471975512 effort=100 velocity=1.5; origin xyz=0 0 0.1105 rpy=0 0 0 -> xyz=0 0 0.05 rpy=0 0 0
- joint L2: axis 0 0 1 -> 0 1 0; limit lower=-2.530881 upper=-0.05890486 effort=300 velocity=3 -> lower=-1.3194689145 upper=1.5707963268 effort=100 velocity=1.5; origin xyz=0.0234207210610375 0 0 rpy=-1.5707963267949 0 0 -> xyz=0.047 0 0.135 rpy=0 0 0
- joint L3: axis 0 0 1 -> 0 1 0; limit lower=1.88261685 upper=5.02423568 effort=300 velocity=3 -> lower=-1.5707963268 upper=1.2566370614 effort=100 velocity=1.5; origin xyz=0.18 0 0 rpy=3.14159265358979 0 0 -> xyz=0 0 0.110 rpy=0 0 0
- joint L4: axis 0 0 1 -> 1 0 0; limit lower=-1.8407944 upper=1.8407944 effort=300 velocity=3 -> lower=-4.7123889804 upper=4.7123889804 effort=100 velocity=1.5; origin xyz=-0.0435 0.17635 0 rpy=1.5707963267949 -1.5707963267949 0 -> xyz=0 0 0.026 rpy=0 0 0
- joint L5: axis 0 0 1 -> 0 1 0; limit lower=-1.57079633 upper=1.57079633 effort=300 velocity=3 -> lower=-1.8849555922 upper=1.8849555922 effort=100 velocity=1.5; origin xyz=0 0 0 rpy=-1.5707963267949 0 0 -> xyz=0.1175 0 0 rpy=0 0 0
- joint L6: axis 0 0 1 -> 1 0 0; limit lower=0.0 upper=6.28318531 effort=300 velocity=3 -> (none); origin xyz=0 0.0628 0 rpy=1.5707963267949 0 0 -> xyz=0.0268 0 0 rpy=0 0 0; type revolute -> continuous
- joint base_joint: origin xyz=0.0 0.0 0.00 rpy=0 0 0 -> xyz=0 0 0 rpy=0 0 0
